Commit message: Turned joint8 into a mimic joint for piper x

File: src/piper_x_description/urdf/piper_x_description.urdf (robot description, URDF)
Before this commit: robot piper_x, 7 links, 6 joints
Links:
- added link link7, mass 0.0; collision mesh filename=package://piper_x_description/meshes/dae/joint7.dae; visual mesh filename=package://piper_x_description/meshes/dae/joint7.dae
- added link link8, mass 0.0264822021416248; collision mesh filename=package://piper_x_description/meshes/dae/joint8.dae; visual mesh filename=package://piper_x_description/meshes/dae/joint8.dae
Joints:
- added joint joint7: type prismatic, parent link6, child link7, origin xyz=0 0 0.13503 rpy=1.5708 0 1.5708, axis 0 0 -1, limit lower=0 upper=0.05 effort=100 velocity=1
- added joint joint8: type prismatic, parent link6, child link8, origin xyz=0 0 0.13503 rpy=-1.5708 0 1.5708, axis 0 0 1, limit lower=-0.05 upper=0 effort=100 velocity=1, mimic joint=joint7 multiplier=-1

File: src/piper_x_description/urdf/piper_x_description.xacro (robot description, xacro)
@@ -461,4 +461,5 @@
         <axis xyz="0 0 1" />
         <limit lower="-0.05" upper="0" effort="100" velocity="1" />
+        <mimic joint="joint7" multiplier="-1" />
     </joint>
 <!-- controller -->

File: src/piper_x_description/urdf/piper_x_description_gazebo.xacro (robot description, xacro)
@@ -461,4 +461,5 @@
         <axis xyz="0 0 1" />
         <limit lower="-0.05" upper="0" effort="100" velocity="1" />
+        <mimic joint="joint7" multiplier="-1" />
     </joint>
   <!-- <gazebo reference="base_link">

File: src/piper_x_description/urdf/piper_x_description_with_teach.urdf (robot description, URDF)
Before this commit: robot piper_x, 9 links, 8 joints
Joints:
- joint joint8: mimic (none) -> joint=joint7 multiplier=-1
